File: pif_fpga/pif_fpga.sch (KiCad schematic (older format))
At the start: 7 parts, among them P1 CONN_02X20, P2 CONN_01X18

Commit message: changed connector to Hirose DF12
Parts:
- P1: footprint pif_fpga:Amphenol_MezzoStak-10106813_2x20x0.5mm -> pif_fpga:Hirose_DF12A-40DS-0.5V_2x20_P0.50mm_Vertical
Changed lines of the file:
@@
 F 0 "P1" H 1450 7100 50  0000 C CNN
 F 1 "CONN_02X20" V 1500 6050 50  0000 C CNN
-F 2 "pif_fpga:Amphenol_MezzoStak-10106813_2x20x0.5mm" H 1450 5100 50  0001 C CNN
+F 2 "pif_fpga:Hirose_DF12A-40DS-0.5V_2x20_P0.50mm_Vertical" H 1450 5100 50  0001 C CNN
 F 3 "" H 1450 5100 50  0000 C CNN
 	1    1450 6050
