File: pif_adapter/pif_adapter.sch (KiCad schematic (older format))
At the start: 11 parts, among them P1 Conn_02x20_Odd_Even, P10 Conn_01x01, P11 Conn_01x01, P2 PIF-NUS, P3 Conn_01x01, P4 Conn_01x01, P5 Conn_01x01, P6 Conn_01x01, P7 Conn_01x01, P8 Conn_01x01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

Commit message: changed connector to Hirose DF12
Parts:
- P1: footprint pif_adapter:Amphenol_MezzoStak-10106813_2x20x0.5mm -> pif_adapter:Hirose_DF12D-40DP-0.5V_2x20_P0.50mm_Vertical
Changed lines of the file:
@@
 F 0 "P1" H 9350 4867 50  0000 C CNN
 F 1 "Conn_02x20_Odd_Even" H 9350 4776 50  0000 C CNN
-F 2 "pif_adapter:Amphenol_MezzoStak-10106813_2x20x0.5mm" H 9300 3750 50  0001 C CNN
+F 2 "pif_adapter:Hirose_DF12D-40DP-0.5V_2x20_P0.50mm_Vertical" H 9300 3750 50  0001 C CNN
 F 3 "~" H 9300 3750 50  0001 C CNN
 	1    9300 3750
